Commit message: Add inertial and collision tags to URDF for gazebo

File: workspace/src/crater_bot/description/bodies/center_chassis.xacro (robot description, xacro)
@@ -2,4 +2,9 @@
 <robot xmlns:xacro="http://www.ros.org/wiki/xacro">
     <link name="compute_box">
+        <inertial>
+            <origin xyz="0.0 0.0 0.0" rpy="0.0 0.0 0.0"/>
+            <mass value="0.0"/>
+            <inertia ixx="0.0" ixy="0.0" ixz="0.0" iyy="0.0" iyz="0.0" izz="0.0"/>
+        </inertial>
         <visual name="compute_box_body">
             <geometry>
@@ -15,4 +20,15 @@
             <material name="orange" />
         </visual>
+        <collision>
+            <geometry>
+                <box size="${chassis_x} ${chassis_y} ${chassis_z}"/>
+            </geometry>
+        </collision>
+        <collision>
+            <origin xyz="${compute_rod_x} 0 ${compute_rod_z}" rpy="${pi/2} 0 0"/>
+            <geometry>
+                <cylinder length="${compute_rod_length}" radius="${compute_rod_radius}" />
+            </geometry>
+        </collision>
     </link>
 </robot>

File: workspace/src/crater_bot/description/bodies/lower_front_suspension.xacro (robot description, xacro)
@@ -8,4 +8,10 @@
             <origin xyz="${reflect*length/3} 0 -${length/3}" rpy="0 ${angle} 0" />
         </visual>
+        <collision>
+            <geometry>
+                <box size="${length} 0.01 0.02" />
+            </geometry>
+            <origin xyz="${reflect*length/3} 0 -${length/3}" rpy="0 ${angle} 0" />
+        </collision>
     </xacro:macro>
     <xacro:macro name="front_lower_suspension" params="prefix reflect offset_angle">

File: workspace/src/crater_bot/description/bodies/upper_suspension.xacro (robot description, xacro)
@@ -10,4 +10,10 @@
                 <material name="white"/>
             </visual>
+            <collision>
+                <origin xyz="${front_length/2} 0 0" />
+                <geometry>
+                    <box size="${front_length} 0.01 0.02"/>
+                </geometry>
+            </collision>
         </link>
         <joint name ="base_to_${prefix}_base_arm_front" type="fixed">
@@ -24,4 +30,10 @@
                 <material name="white"/>
             </visual>
+            <collision>
+                <origin xyz="${front_length/2} 0 0" />
+                <geometry>
+                    <box size="${front_length} 0.01 0.02"/>
+                </geometry>
+            </collision>
         </link>
         <joint name ="base_to_${prefix}_base_arm_back" type="fixed">

File: workspace/src/crater_bot/description/bodies/wheel.xacro (robot description, xacro)
@@ -9,4 +9,14 @@
                 <material name="blue" />
             </visual>
+            <collision>
+                <geometry>
+                    <cylinder radius="0.05" length="0.04" />
+                </geometry>
+            </collision>
+            <inertial>
+                <origin xyz="0 0 0" rpy="0 0 0"/>
+                <mass value="0.5"/>
+                <inertia ixx="0.001" ixy="0.0" ixz="0.0" iyy="0.001" iyz="0.0" izz="0.001"/>
+            </inertial>
         </link>
         <joint name="${prefix}_wheel_to_lower_suspension" type="continuous">
