Commit message: Include dummy and base link with inertia

File: workspace/src/crater_bot/description/crater_core.xacro (robot description, xacro)
@@ -25,11 +25,22 @@
     <xacro:include filename="bodies/lower_front_suspension.xacro" />
     <xacro:include filename="bodies/wheel.xacro" />
-    <!-- Center Frame of Reference -->
-    <link name="base_link" />
+    <!-- Dummy + Base Links -->
+    <link name="dummy" />
+    <link name="base_link">
+        <inertial>
+            <origin xyz="0 0 0.017"/>
+            <mass value="1.2"/>
+            <inertia ixx="0.0001873" ixy="0" ixz="0" iyy="0.000055" iyz="0" izz="0.0002283" />
+        </inertial>
+    </link>
+    <joint name="dummy_joint" type="fixed">
+        <parent link="dummy"/>
+        <child link="base_link"/>
+    </joint>
     <!-- Link body to origin rod  -->
-    <joint name="compute_box_joint" type="fixed">
+    <joint name="base_link_to_chassis" type="fixed">
         <parent link="base_link" />
         <child link="compute_box" />
-        <origin xyz="0 0 0.2" />
+        <origin xyz="0 0 1" />
     </joint>
     <!-- Add arm bases to compute rod -->

Commit message: Add ros2_control to enable remote control

File: workspace/src/crater_bot/description/crater_core.xacro (robot description, xacro)
@@ -53,9 +53,9 @@
     <!-- 3 Left Wheels -->
     <xacro:wheel parent="left_front_lower_susp" prefix="LF" reflect="1" offset_x="0.065" offset_z="-0.06"/>
-    <xacro:wheel parent="left_front_lower_susp" prefix="LM" reflect="1" offset_x="-0.065" offset_z="-0.06"/>
-    <xacro:wheel parent="left_base_arm_back" prefix="LR" reflect="1" offset_x="${-back_length}" offset_z="0"/>
+    <!-- <xacro:wheel parent="left_front_lower_susp" prefix="LM" reflect="1" offset_x="-0.065" offset_z="-0.06"/> -->
+    <!-- <xacro:wheel parent="left_base_arm_back" prefix="LR" reflect="1" offset_x="${-back_length}" offset_z="0"/> -->
     <!-- 3 Right Wheels -->
     <xacro:wheel parent="right_front_lower_susp" prefix="RF" reflect="-1" offset_x="0.065" offset_z="-0.06"/>
-    <xacro:wheel parent="right_front_lower_susp" prefix="RM" reflect="-1" offset_x="-0.065" offset_z="-0.06"/>
-    <xacro:wheel parent="right_base_arm_back" prefix="RR" reflect="-1" offset_x="${-back_length}" offset_z="0"/>
+    <!-- <xacro:wheel parent="right_front_lower_susp" prefix="RM" reflect="-1" offset_x="-0.065" offset_z="-0.06"/> -->
+    <!-- <xacro:wheel parent="right_base_arm_back" prefix="RR" reflect="-1" offset_x="${-back_length}" offset_z="0"/> -->
 </robot>

File: workspace/src/crater_bot/description/ros2_control.xacro (robot description, xacro)
@@ -12,8 +12,13 @@
         </joint>
     </xacro:macro>
+    <xacro:macro name="odrive" params="name id">
+        <joint name="${name}_wheel_to_lower_suspension">
+            <param name="node_id">${id}</param>
+        </joint>
+    </xacro:macro>
     <xacro:macro name="diffbot_ros2_control" params="name use_mock_hardware">
         <ros2_control name="${name}" type="system">
             <!-- Simulation Config -->
-            <xacro:if value="${use_mock_hardware}">
+            <!-- <xacro:if value="${use_mock_hardware}">
                 <hardware>
                     <plugin>gz_ros2_control/GazeboSimSystem</plugin>
@@ -26,17 +31,17 @@
                 <xacro:r2c_wheel name="RM" />
                 <xacro:r2c_wheel name="RR" />
-            </xacro:if>
+            </xacro:if> -->
             <!-- Crater Config -->
             <xacro:unless value="${use_mock_hardware}">
                 <hardware>
                     <plugin>odrive_ros2_control_plugin/ODriveHardwareInterface</plugin>
-                    <param name="can">can1</param>
+                    <param name="can">can0</param>
                 </hardware>
-                <joint name="RF_wheel_to_lower_suspension">
-                    <param name="node_id">0</param>
-                </joint>
-                <joint name="LF_wheel_to_lower_suspension">
-                    <param name="node_id">1</param>
-                </joint>
+                <xacro:odrive name="LF" id="1" />
+                <!-- <xacro:odrive name="LM" id="2" /> -->
+                <!-- <xacro:odrive name="LR" id="3" /> -->
+                <xacro:odrive name="RF" id="2" />
+                <!-- <xacro:odrive name="RM" id="4" /> -->
+                <!-- <xacro:odrive name="RR" id="5" /> -->
             </xacro:unless>
             <!-- <xacro:if value="${use_mock_hardware}">
